File: Prototyping Board/prototype.brd (EAGLE design)
At the start: 160 x 100 mm, 35 parts

Commit message: first version of the board
Parts:
- removed LD1, LD2, LD3, LD4, LD5: PL006-WCR12, led:SOT23
- removed R1, R10, R11, R12, R13, R14, R15, R16, R17, R18, R19, R2, R20, R21, R22, R23, R24, R25, R26, R27, R28, R29, R3, R30, R4, R5, R6, R7, R8, R9: (no value), resistor:M0805
- added E$1, E$10, E$12, E$13, E$14, E$2, E$3, E$4, E$5, E$6, E$7, E$8, E$9: (no value), 80_50:BB_TSSOP_0650
- added E$11: (no value), dp_devices:BB_QFP_050_065_BREAKOUT_BOARD
- added E$15: (no value), dp_devices:BB_QFP_080_050_BREAKOUT_BOARD
- added E$16, E$17, E$18, E$19, E$20, E$21, E$22, E$23, E$24, E$25, E$26, E$27, E$28: (no value), 80_50:BB_SOIC
- added E$192, E$193, E$194, E$195, E$196, E$197, E$198, E$199, E$200, E$201, E$202, E$203, E$204, E$205, E$206, E$207, E$208, E$209, E$210, E$211, E$212, E$213, E$214, E$215, E$216, E$217, E$218, E$219, E$220, E$35, E$36, E$37, E$38, E$517, E$518, E$519, E$54, E$55, E$56, E$57, E$58, E$59, E$60, E$61: (no value), 80_50:BB_RC0805
- added E$250, E$251, E$252, E$254, E$255, E$31, E$32, E$33, E$39, E$40: (no value), 80_50:BB_SOT23-6
- added E$258, E$29: (no value), 80_50:BB_XTAL
- added E$260, E$34: (no value), 80_50:BB_SW
- added E$30: (no value), 80_50:PROTO_THROUGH
Other:
- board size 160 x 100 mm -> 80 x 100 mm

Commit message: added kais wishes :)
Parts:
- removed E$192, E$193, E$194, E$197, E$198, E$199, E$200, E$201, E$202, E$204, E$205, E$206, E$207, E$208, E$209, E$210, E$211, E$212, E$216, E$217, E$35, E$37, E$38, E$517, E$518: (no value), 80_50:BB_RC0805
- removed E$39, E$40: (no value), 80_50:BB_SOT23-6
- E$11: device dp_devices:BB_QFP_050_065_BREAKOUT_BOARD -> 80_50:BB_QFP_080_050_BREAKOUT_BOARD
- E$15: device dp_devices:BB_QFP_080_050_BREAKOUT_BOARD -> 50_65:BB_QFP_050_065_BREAKOUT_BOARD
- E$28: device 80_50:BB_SOIC -> 80_50:BB_SOT23-6
- E$32: device 80_50:BB_SOT23-6 -> 80_50:VCC_GND
- E$33: device 80_50:BB_SOT23-6 -> 80_50:SUBD9
- E$36: device 80_50:BB_RC0805 -> 80_50:BB_TSSOP_0650
- moved E$16 76.2 mm to (6.50, 52.6), turned to 90 degrees
- moved E$17 72.5 mm to (9.10, 52.6), turned to 90 degrees
- moved E$18 68.9 mm to (11.7, 52.6), turned to 90 degrees
- moved E$19 65.3 mm to (14.3, 52.6), turned to 90 degrees
- moved E$11 61.7 mm to (21.6, 20.3)
- moved E$20 61.7 mm to (16.9, 52.6), turned to 90 degrees
- moved E$15 61.5 mm to (18.4, 81.9)
- moved E$250 59.1 mm to (72.8, 33.1), turned to 270 degrees
- moved E$21 58.1 mm to (19.5, 52.6), turned to 90 degrees
- moved E$33 55.9 mm to (2.54, 52.1), turned to 90 degrees
- moved E$22 54.4 mm to (22.1, 52.6), turned to 90 degrees
- moved E$251 54.1 mm to (72.8, 42.2), turned to 90 degrees
- moved E$23 50.8 mm to (24.7, 52.6), turned to 90 degrees
- moved E$24 47.3 mm to (27.3, 52.6), turned to 90 degrees
- moved E$519 45.2 mm to (61.4, 35.4), turned to 90 degrees
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Connections:
- new net S$14: E$32.P$2
Routing:
- net S$5: track 0.00 -> 65.4 mm, vias 0 -> 2
- net S$14: track 0.00 -> 59.1 mm, vias 0 -> 2
- net S$11: track 0.00 -> 40.6 mm, vias 0 -> 1
- net S$13: track 0.00 -> 15.2 mm, vias 0 -> 1
- added copper zone on layer 16, net GND

Commit message: added mosfets
Parts:
- removed E$258: (no value), 80_50:BB_XTAL
- added E$35: (no value), 80_50:BB_XTAL
- added E$37, E$38, E$39: (no value), 80_50:TO-263
- added E$40, E$41, E$42, E$43, E$44, E$45: (no value), 80_50:TO-252
- added MAX3232: (no value), maxim:SO16
- moved E$29 42.1 mm to (42.5, 90.8)
Connections:
- net S$14: now also E$32.P$24; no longer E$32.P$2
Routing:
- net S$14: track 59.1 -> 59.7 mm
Changed lines of the file:
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@@
 <layer number="19" name="Unrouted" color="6" fill="1" visible="yes" active="yes"/>
 <layer number="20" name="Dimension" color="15" fill="1" visible="yes" active="yes"/>
-<layer number="21" name="tPlace" color="7" fill="1" visible="yes" active="yes"/>
-<layer number="22" name="bPlace" color="7" fill="1" visible="no" active="yes"/>
-<layer number="23" name="tOrigins" color="15" fill="1" visible="yes" active="yes"/>
-<layer number="24" name="bOrigins" color="15" fill="1" visible="no" active="yes"/>
-<layer number="25" name="tNames" color="7" fill="1" visible="yes" active="yes"/>
-<layer number="26" name="bNames" color="7" fill="1" visible="no" active="yes"/>
-<layer number="27" name="tValues" color="7" fill="1" visible="yes" active="yes"/>
-<layer number="28" name="bValues" color="7" fill="1" visible="no" active="yes"/>
+<layer number="21" name="tPlace" color="7" fill="1" visible="no" active="yes"/>
+<layer number="22" name="bPlace" color="7" fill="1" visible="yes" active="yes"/>
+<layer number="23" name="tOrigins" color="15" fill="1" visible="no" active="yes"/>
+<layer number="24" name="bOrigins" color="15" fill="1" visible="yes" active="yes"/>
+<layer number="25" name="tNames" color="7" fill="1" visible="no" active="yes"/>
+<layer number="26" name="bNames" color="7" fill="1" visible="yes" active="yes"/>
+<layer number="27" name="tValues" color="7" fill="1" visible="no" active="yes"/>
+<layer number="28" name="bValues" color="7" fill="1" visible="yes" active="yes"/>
 <layer number="29" name="tStop" color="7" fill="3" visible="no" active="yes"/>
 <layer number="30" name="bStop" color="7" fill="6" visible="yes" active="yes"/>
@@
 <layer number="49" name="Reference" color="7" fill="1" visible="no" active="yes"/>
 <layer number="50" name="dxf" color="7" fill="1" visible="no" active="yes"/>
-<layer number="51" name="tDocu" color="7" fill="1" visible="yes" active="yes"/>
+<layer number="51" name="tDocu" color="7" fill="1" visible="no" active="yes"/>
 <layer number="52" name="bDocu" color="7" fill="1" visible="no" active="yes"/>
 <layer number="91" name="Nets" color="2" fill="1" visible="no" active="no"/>
@@
 <layer number="97" name="Info" color="7" fill="1" visible="no" active="no"/>
 <layer number="98" name="Guide" color="6" fill="1" visible="no" active="no"/>
+<layer number="99" name="SpiceOrder" color="5" fill="1" visible="no" active="no"/>
 </layers>
 <board>
@@
 <param name="mtCopper" value="0.035mm 0.035mm 0.035mm 0.035mm 0.035mm 0.035mm 0.035mm 0.035mm 0.035mm 0.035mm 0.035mm 0.035mm 0.035mm 0.035mm 0.035mm 0.035mm"/>
 <param name="mtIsolate" value="1.5mm 0.15mm 0.2mm 0.15mm 0.2mm 0.15mm 0.2mm 0.15mm 0.2mm 0.15mm 0.2mm 0.15mm 0.2mm 0.15mm 0.2mm"/>
-<param name="mdWireWire" value="0.2mm"/>
+<param name="mdWireWire" value="8mil"/>
 <param name="mdWirePad" value="8mil"/>
 <param name="mdWireVia" value="8mil"/>
@@
 <param name="rlMinPadBottom" value="10mil"/>
 <param name="rlMaxPadBottom" value="20mil"/>
-<param name="rlMinViaOuter" value="2mil"/>
+<param name="rlMinViaOuter" value="4mil"/>
 <param name="rlMaxViaOuter" value="20mil"/>
 <param name="rlMinViaInner" value="8mil"/>
@@
 <element name="E$254" library="80_50" package="BB_SOT23-6" value="" x="72.8" y="46.8" rot="R90"/>
 <element name="E$255" library="80_50" package="BB_SOT23-6" value="" x="72.8" y="37.7" rot="R90"/>
-<element name="E$258" library="80_50" package="BB_XTAL" value="" x="41.995" y="90.96" rot="R270"/>
 <element name="E$260" library="80_50" package="BB_SW" value="" x="52.08" y="33.5"/>
 <element name="E$519" library="80_50" package="BB_RC0805" value="" x="61.425" y="35.425" rot="R90"/>
@@
 <element name="E$60" library="80_50" package="BB_RC0805" value="" x="46.15" y="95.55" rot="R90"/>
 <element name="E$61" library="80_50" package="BB_RC0805" value="" x="40.95" y="78" rot="R90"/>
-<element name="E$29" library="80_50" package="BB_XTAL" value="" x="42.9" y="48.75" rot="R270"/>
 <element name="E$31" library="80_50" package="BB_SOT23-6" value="" x="52.65" y="46.15" rot="R270"/>
 <element name="E$34" library="80_50" package="BB_SW" value="" x="52.73" y="51.2"/>
@@
 <element name="E$11" library="80_50" package="BB_QFP_080_050_BREAKOUT_BOARD" value="" x="21.59" y="20.32"/>
 <element name="E$15" library="50_65" package="BB_QFP_050_065_BREAKOUT_BOARD" value="" x="18.415" y="81.915"/>
+<element name="E$29" library="80_50" package="BB_XTAL" value="" x="42.545" y="90.805" rot="R270"/>
+<element name="E$35" library="80_50" package="BB_XTAL" value="" x="42.545" y="48.895" rot="R270"/>
+<element name="E$37" library="80_50" package="TO-263" value="" x="48.26" y="41.91" rot="MR0"/>
+<element name="E$38" library="80_50" package="TO-263" value="" x="60.96" y="41.91" rot="MR0"/>
+<element name="E$39" library="80_50" package="TO-263" value="" x="73.66" y="41.91" rot="MR0"/>
+<element name="E$40" library="80_50" package="TO-252" value="" x="41.91" y="86.36" rot="MR0"/>
+<element name="E$41" library="80_50" package="TO-252" value="" x="68.58" y="29.21" rot="MR90"/>
+<element name="E$42" library="80_50" package="TO-252" value="" x="54.61" y="29.21" rot="MR270"/>
+<element name="E$43" library="80_50" package="TO-252" value="" x="41.91" y="71.12" rot="MR0"/>
+<element name="E$44" library="80_50" package="TO-252" value="" x="34.29" y="49.53" rot="MR0"/>
+<element name="E$45" library="80_50" package="TO-252" value="" x="25.4" y="49.53" rot="MR0"/>
+<element name="MAX3232" library="maxim" package="SO16" value="" x="11.43" y="52.07" smashed="yes" rot="MR270">
+<attribute name="VALUE" x="12.065" y="56.134" size="1.27" layer="28" ratio="10" rot="MR270"/>
+<attribute name="NAME" x="12.319" y="55.372" size="1.27" layer="26" ratio="10" rot="MR270"/>
+</element>
 </elements>
 <signals>
@@
 <wire x1="5.08" y1="67.31" x2="1.27" y2="67.31" width="0.8128" layer="16"/>
 <via x="34.925" y="66.675" extent="1-16" drill="0.8" shape="square"/>
-<contactref element="E$32" pad="P$2"/>
-<wire x1="48.895" y1="66.675" x2="36.83" y2="66.675" width="0.8128" layer="16"/>
 <wire x1="36.83" y1="66.675" x2="34.925" y2="66.675" width="0.8128" layer="16"/>
 <wire x1="36.83" y1="62.23" x2="36.83" y2="66.675" width="0.8128" layer="16"/>
+<wire x1="36.83" y1="62.23" x2="48.895" y2="62.23" width="0.8128" layer="16"/>
+<contactref element="E$32" pad="P$24"/>
+<wire x1="48.895" y1="62.23" x2="48.895" y2="61.595" width="0.8128" layer="16"/>
 </signal>
 <signal name="GND">

Commit message: minor changes
Routing:
- net GND: track 0.00 -> 20.4 mm
Changed lines of the file:
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@@
 <setting verticaltext="up"/>
 </settings>
-<grid distance="1.27" unitdist="mm" unit="mm" style="lines" multiple="1" display="yes" altdistance="0.635" altunitdist="mm" altunit="mm"/>
+<grid distance="1.27" unitdist="mm" unit="mm" style="lines" multiple="1" display="yes" altdistance="0.1" altunitdist="mm" altunit="mm"/>
 <layers>
 <layer number="1" name="Top" color="4" fill="1" visible="no" active="yes"/>
@@
 <via x="40.005" y="36.83" extent="1-16" drill="0.8" shape="square"/>
 <via x="40.005" y="1.905" extent="1-16" drill="0.8" shape="square"/>
-<polygon width="0.8128" layer="16">
+<polygon width="0.8128" layer="16" isolate="0.3048">
 <vertex x="-0.635" y="100.965"/>
 <vertex x="80.645" y="100.965"/>
@@
 </polygon>
 <via x="3.175" y="1.905" extent="1-16" drill="0.8" shape="square"/>
+<wire x1="47.625" y1="95.885" x2="53.34" y2="95.885" width="0.6096" layer="16"/>
+<wire x1="47.625" y1="60.325" x2="52.07" y2="60.325" width="0.6096" layer="16"/>
+<wire x1="47.625" y1="70.485" x2="52.705" y2="70.485" width="0.6096" layer="16"/>
+<wire x1="60.7" y1="25" x2="60.6" y2="25" width="0.6096" layer="16"/>
+<wire x1="60.6" y1="25" x2="60.6" y2="23.6" width="0.6096" layer="16"/>
+<wire x1="61.9" y1="6.8" x2="61.9" y2="5.7" width="0.6096" layer="16"/>
+<wire x1="68.5" y1="25.1" x2="68.4" y2="25.1" width="0.6096" layer="16"/>
+<wire x1="68.4" y1="25.1" x2="68.4" y2="23.6" width="0.6096" layer="16"/>
+<wire x1="69.7" y1="6.8" x2="69.7" y2="5.8" width="0.6096" layer="16"/>
+<wire x1="47.625" y1="70.485" x2="47.625" y2="60.325" width="0" layer="19" extent="16-16"/>
+<wire x1="60.6" y1="25" x2="40.005" y2="36.83" width="0" layer="19" extent="16-16"/>
+<wire x1="68.4" y1="25.1" x2="60.7" y2="25" width="0" layer="19" extent="16-16"/>
+<wire x1="61.9" y1="6.8" x2="60.6" y2="23.6" width="0" layer="19" extent="16-16"/>
 </signal>
 </signals>
